File: Hardware/template/template.kicad_pcb (KiCad board)
At the start: 4 copper layers, 0 parts

Commit message: basic circuit to test that the pipe line works
Parts:
- added BT1: Battery, Battery:BatteryHolder_LINX_BAT-HLD-012-SMT, F.Cu at (140.8, 100.4)
- added D1: LED, LED_SMD:LED_0805_2012Metric, F.Cu at (130.2, 100.6)
- added H1: MountingHole, MountingHole:MountingHole_3.2mm_M3_DIN965_Pad, F.Cu at (131.8, 91.2)
- added H2: MountingHole, MountingHole:MountingHole_3.2mm_M3_DIN965_Pad, F.Cu at (149.6, 91.2)
- added H3: MountingHole, MountingHole:MountingHole_3.2mm_M3_DIN965_Pad, F.Cu at (131.8, 109.0)
- added H4: MountingHole, MountingHole:MountingHole_3.2mm_M3_DIN965_Pad, F.Cu at (149.6, 109.0)
- added R1: R, Resistor_SMD:R_0805_2012Metric, F.Cu at (151.2, 100.6)
Routing:
- net Net-(D1-A): track 0.00 -> 27.2 mm
- net /+V: track 0.00 -> 25.1 mm
- net /-V: track 0.00 -> 1.06 mm, vias 0 -> 37
- added copper zone on In2.Cu, net /-V
Other:
- board outline added: 25 x 25 mm
- board text added: "TEST_BOARD DELETE"
