File: Hardware/template/template.kicad_sch (KiCad schematic)
At the start: 0 parts

Commit message: basic circuit to test that the pipe line works
Parts:
- added BT1: Battery, Battery:BatteryHolder_LINX_BAT-HLD-012-SMT, symbol Device:Battery
- added D1: LED, LED_SMD:LED_0805_2012Metric, symbol Device:LED
- added H1, H2, H3, H4: MountingHole, MountingHole:MountingHole_3.2mm_M3_DIN965_Pad, symbol Mechanical:MountingHole
- added R1: R, Resistor_SMD:R_0805_2012Metric, symbol Device:R
Connections:
- new net: D1.2 (A), R1.2
- new net +V: BT1.1 (+), R1.1
- new net -V: BT1.2 (-), D1.1 (K)
