File: Hardware/template/template.kicad_sch (KiCad schematic)
At the start: 7 parts

Commit message: added boxes
Other:
- note added: "CIRCUIT"
- note added: "MOUNTING HOLES"
- moved on the sheet: BT1, D1, H1, H2, H3, H4, R1
